File: NRF24-zero-SHIM.sch (EAGLE design)
At the start: 36 parts

Commit message: Fixed document description.
Other:
- note added: "Pi Zero sized NRF24-SHIM for Pi's 40-pin extension slot (c) Andriy Golovnya"
- note removed: "Double-mount NRF24-SHIM for Pi's 40-pin extension slot (c) Andriy Golovnya"
Changed lines of the file:
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@@
 <text x="256.54" y="7.62" size="2.54" layer="94">1.0</text>
 <text x="198.12" y="7.62" size="2.54" layer="94">PI-NRF24ZS-0010</text>
-<text x="165.1" y="25.4" size="2.54" layer="94">Double-mount NRF24-SHIM for Pi's 40-pin extension slot
+<text x="165.1" y="25.4" size="2.54" layer="94">Pi Zero sized NRF24-SHIM for Pi's 40-pin extension slot
 (c) Andriy Golovnya</text>
 <text x="33.02" y="147.32" size="2.54" layer="94">NRF24 connectors</text>
